File: nPNP_Feeder/Electrical/ConnectorHolder/ConnectorHolderPCB_V0.3.brd (EAGLE design)
At the start: 420 x 13 mm, 27 parts, among them J21 1734366-1, J22 1734366-1, J23 1734366-1, J24 1734366-1, J25 1734366-1, J26 1734366-1, J27 1734366-1, J28 1734366-1, J29 1734366-1, J30 1734366-1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

Commit message: Added BOM, schematic as pdf and PCB as image
Parts:
- removed U$2: (no value), PNPFeeder:LOGO
- U$1: device PNPFeeder:LOGO -> PNPFeeder:NPNP_LARGE_NOTEXT
- moved U$1 0.10 mm to (-382.5, -1.30), flipped to the bottom
Other:
- board text added: "FEEDER BRACKET"
- board text removed: "FeederBracket"
Changed lines of the file:
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@@
 <drawing>
 <settings>
-<setting alwaysvectorfont="no"/>
+<setting alwaysvectorfont="yes"/>
 <setting verticaltext="up"/>
 </settings>
@@
 <circle x="-376" y="-1.3" radius="2.2" width="0.254" layer="20"/>
 <circle x="22" y="-1.3" radius="2.2" width="0.254" layer="20"/>
-<text x="-382.61" y="-1.6" size="0.5" layer="22" ratio="15" rot="MR0" align="center">V0.1 - 01/07/2021</text>
-<text x="-382.58" y="-0.78" size="0.7" layer="22" ratio="15" rot="MR0" align="center">FeederBracket</text>
+<text x="-380.61" y="-6.3" size="0.85" layer="22" ratio="15" rot="MR0" align="center">V0.1 - 01/07/2021</text>
+<text x="-380.58" y="-5.08" size="1.016" layer="22" ratio="15" rot="MR0" align="center">FEEDER BRACKET</text>
 <text x="30.5" y="2.5" size="0.6096" layer="22" ratio="15" rot="MR0" align="center-right">VCC</text>
 <text x="30.5" y="0.5" size="0.6096" layer="22" ratio="15" rot="MR0" align="center-right">GND</text>
@@
 <attribute name="VALUE" x="29" y="2.5" size="0.0254" layer="28" rot="MR90"/>
 </element>
-<element name="U$1" library="PNPFeeder" package="LOGO" value="" x="-382.6" y="-1.3" smashed="yes"/>
-<element name="U$2" library="PNPFeeder" package="LOGO" value="" x="15.8" y="-1.3" smashed="yes"/>
 <element name="PAD5" library="wirepad" library_urn="urn:adsk.eagle:library:412" package="SMD1,27-2,54" package3d_urn="urn:adsk.eagle:package:30839/1" value="" x="29" y="-5.5" smashed="yes" rot="MR270">
 <attribute name="POPULARITY" value="15" x="23" y="-1.5" size="1.778" layer="28" rot="MR270" display="off"/>
 <attribute name="VALUE" x="29" y="-5.5" size="0.0254" layer="28" rot="MR270"/>
 </element>
+<element name="U$1" library="PNPFeeder" package="NPNP_LARGE_NOTEXT" value="" x="-382.5" y="-1.3" smashed="yes" rot="MR0"/>
 </elements>
 <signals>
@@
 </signals>
 <mfgpreviewcolors>
-<mfgpreviewcolor name="soldermaskcolor" color="0xC8008000"/>
+<mfgpreviewcolor name="soldermaskcolor" color="0xC8000000"/>
 <mfgpreviewcolor name="silkscreencolor" color="0xFFFEFEFE"/>
 <mfgpreviewcolor name="backgroundcolor" color="0xFF282828"/>
